File: Hardware/WRFL_User_Interface.sch (KiCad schematic (older format))
At the start: 13 parts, among them P16 2x3_2_54_RA_MALE, Q3 SI1012CR, SW1 TSA12110, SW2 EN11-HSB, SW3 TSA12110, U9 S25FL216K0PMFI040

Commit message: MCU function assignment
BT RTS/CTS as test points,
BT reset GPIO option
Launchpad header pin function assignment (for ERC check)
Power symbols corrections
Connections:
- net LCD_D_C renamed LCD_C_D
Changed lines of the file:
@@
-EESchema Schematic File Version 2  date Tuesday, October 15, 2013 09:37:22 AM
+EESchema Schematic File Version 2  date Tuesday, October 22, 2013 02:02:38 PM
 LIBS:power
 LIBS:device
@@
 Sheet 4 6
 Title ""
-Date "15 oct 2013"
+Date "22 oct 2013"
 Rev ""
 Comp "Nightmechanic"
@@
 LCD_CS
 Text GLabel 2150 2800 3    60   Input ~ 0
-LCD_D_C
+LCD_C_D
 Text GLabel 2350 2800 3    60   Input ~ 0
 GEN_SSI_TX
@@
 GEN_SSI_CLK
 $Comp
-L VDD_PERIPH #U13
+L VDD_PERIPH #U049
 U 1 1 5251E2C5
 P 950 3350
-F 0 "#U13" H 950 3550 60  0001 C CNN
+F 0 "#U049" H 950 3550 60  0001 C CNN
 F 1 "VDD_PERIPH" H 950 3450 60  0000 C CNN
 F 2 "~" H 950 3350 60  0000 C CNN
@@
 $EndComp
 $Comp
-L VDD_PERIPH #U16
+L VDD_PERIPH #U050
 U 1 1 5251E301
 P 9300 1550
-F 0 "#U16" H 9300 1750 60  0001 C CNN
+F 0 "#U050" H 9300 1750 60  0001 C CNN
 F 1 "VDD_PERIPH" H 9300 1650 60  0000 C CNN
 F 2 "~" H 9300 1550 60  0000 C CNN
@@
 $EndComp
 $Comp
-L GND #PWR31
+L GND #PWR051
 U 1 1 5251E310
 P 950 4350
-F 0 "#PWR31" H 950 4350 30  0001 C CNN
+F 0 "#PWR051" H 950 4350 30  0001 C CNN
 F 1 "GND" H 950 4280 30  0001 C CNN
 F 2 "" H 950 4350 60  0000 C CNN
@@
 $EndComp
 $Comp
-L GND #PWR32
+L GND #PWR052
 U 1 1 5251E31F
 P 2600 6250
-F 0 "#PWR32" H 2600 6250 30  0001 C CNN
+F 0 "#PWR052" H 2600 6250 30  0001 C CNN
 F 1 "GND" H 2600 6180 30  0001 C CNN
 F 2 "" H 2600 6250 60  0000 C CNN
@@
 $EndComp
 $Comp
-L GND #PWR35
+L GND #PWR053
 U 1 1 5251E32E
 P 4450 5950
-F 0 "#PWR35" H 4450 5950 30  0001 C CNN
+F 0 "#PWR053" H 4450 5950 30  0001 C CNN
 F 1 "GND" H 4450 5880 30  0001 C CNN
 F 2 "" H 4450 5950 60  0000 C CNN
@@
 $EndComp
 $Comp
-L GND #PWR36
+L GND #PWR054
 U 1 1 5251E33D
 P 6500 6400
-F 0 "#PWR36" H 6500 6400 30  0001 C CNN
+F 0 "#PWR054" H 6500 6400 30  0001 C CNN
 F 1 "GND" H 6500 6330 30  0001 C CNN
 F 2 "" H 6500 6400 60  0000 C CNN
@@
 $EndComp
 $Comp
-L GND #PWR34
+L GND #PWR055
 U 1 1 5251E34C
 P 3150 2500
-F 0 "#PWR34" H 3150 2500 30  0001 C CNN
+F 0 "#PWR055" H 3150 2500 30  0001 C CNN
 F 1 "GND" H 3150 2430 30  0001 C CNN
 F 2 "" H 3150 2500 60  0000 C CNN
@@
 $EndComp
 $Comp
-L GND #PWR37
+L GND #PWR056
 U 1 1 5251E35B
 P 7500 2700
-F 0 "#PWR37" H 7500 2700 30  0001 C CNN
+F 0 "#PWR056" H 7500 2700 30  0001 C CNN
 F 1 "GND" H 7500 2630 30  0001 C CNN
 F 2 "" H 7500 2700 60  0000 C CNN
@@
 $EndComp
 $Comp
-L GND #PWR33
+L GND #PWR057
 U 1 1 5251E3CC
 P 2950 4350
-F 0 "#PWR33" H 2950 4350 30  0001 C CNN
+F 0 "#PWR057" H 2950 4350 30  0001 C CNN
 F 1 "GND" H 2950 4280 30  0001 C CNN
 F 2 "" H 2950 4350 60  0000 C CNN
@@
 	9300 2050 8850 2050
 Wire Wire Line
-	9300 1750 9300 1850
-Wire Wire Line
-	9300 1850 9300 2050
-Wire Wire Line
-	9300 2050 9300 2200
+	9300 1750 9300 2200
 Wire Wire Line
 	9300 2200 8850 2200
@@
 $EndComp
 $Comp
-L GND #PWR41
+L GND #PWR058
 U 1 1 5251EA53
 P 10150 2500
-F 0 "#PWR41" H 10150 2500 30  0001 C CNN
+F 0 "#PWR058" H 10150 2500 30  0001 C CNN
 F 1 "GND" H 10150 2430 30  0001 C CNN
 F 2 "" H 10150 2500 60  0000 C CNN
@@
 	10150 1850 10150 1900
 $Comp
-L VDD_PERIPH #U14
+L VDD_PERIPH #U059
 U 1 1 5251EAB9
 P 5950 1150
-F 0 "#U14" H 5950 1350 60  0001 C CNN
+F 0 "#U059" H 5950 1350 60  0001 C CNN
 F 1 "VDD_PERIPH" H 5950 1250 60  0000 C CNN
 F 2 "~" H 5950 1150 60  0000 C CNN
@@
 $EndComp
 Wire Wire Line
-	6700 2050 7300 2050
-Wire Wire Line
-	7300 2050 7650 2050
+	6700 2050 7650 2050
 Wire Wire Line
 	7300 2050 7300 1950
@@
 	6550 6100 6500 6100
 Wire Wire Line
-	6500 6100 6500 6300
-Wire Wire Line
-	6500 6300 6500 6400
+	6500 6100 6500 6400
 Wire Wire Line
 	7350 6100 7450 6100
@@
 	2400 6000 2600 6000
 Wire Wire Line
-	2600 6000 2600 6150
-Wire Wire Line
-	2600 6150 2600 6250
+	2600 6000 2600 6250
 Wire Wire Line
 	2600 6150 1450 6150
@@
 USER_SW
 Wire Wire Line
-	6200 5700 6350 5700
-Wire Wire Line
-	6350 5700 6550 5700
-Wire Wire Line
-	7350 5700 7500 5700
-Wire Wire Line
-	7500 5700 7500 5300
-Wire Wire Line
 	7500 5300 6350 5300
 Wire Wire Line
@@
 Connection ~ 6350 5700
 Wire Wire Line
-	1200 5600 1500 5600
-Wire Wire Line
-	1500 5600 1600 5600
+	1200 5600 1600 5600
 Wire Wire Line
 	4450 5750 4450 5950
 Wire Wire Line
-	4700 5750 4700 6000
-Wire Wire Line
-	4700 6000 4700 6200
+	4700 5750 4700 6200
 Wire Wire Line
 	4700 6000 4950 6000
 Wire Wire Line
-	4200 5750 4200 6000
-Wire Wire Line
-	4200 6000 4200 6200
+	4200 5750 4200 6200
 Wire Wire Line
 	4200 6000 4000 6000
@@
 Connection ~ 4700 6000
 Wire Wire Line
-	3150 6800 4200 6800
-Wire Wire Line
-	4200 6800 4700 6800
+	3150 6800 4700 6800
 Wire Wire Line
 	4700 6800 4700 6700
@@
 $EndComp
 $Comp
-L GND #PWR40
+L GND #PWR060
 U 1 1 52523A67
 P 9800 4700
-F 0 "#PWR40" H 9800 4700 30  0001 C CNN
+F 0 "#PWR060" H 9800 4700 30  0001 C CNN
 F 1 "GND" H 9800 4630 30  0001 C CNN
 F 2 "" H 9800 4700 60  0000 C CNN
@@
 $EndComp
 $Comp
-L GND #PWR39
+L GND #PWR061
 U 1 1 52523A76
 P 8750 4700
-F 0 "#PWR39" H 8750 4700 30  0001 C CNN
+F 0 "#PWR061" H 8750 4700 30  0001 C CNN
 F 1 "GND" H 8750 4630 30  0001 C CNN
 F 2 "" H 8750 4700 60  0000 C CNN
@@
 	9800 4500 9800 4700
 $Comp
-L V_BOOST #U15
+L V_BOOST #U062
 U 1 1 52523B29
 P 8300 4200
-F 0 "#U15" H 8300 4400 60  0001 C CNN
+F 0 "#U062" H 8300 4400 60  0001 C CNN
 F 1 "V_BOOST" H 8300 4300 60  0000 C CNN
 F 2 "~" H 8300 4200 60  0000 C CNN
@@
 $EndComp
 $Comp
-L V_BOOST #U17
+L V_BOOST #U063
 U 1 1 52523B38
 P 10200 4200
-F 0 "#U17" H 10200 4400 60  0001 C CNN
+F 0 "#U063" H 10200 4400 60  0001 C CNN
 F 1 "V_BOOST" H 10200 4300 60  0000 C CNN
 F 2 "~" H 10200 4200 60  0000 C CNN
@@
 $EndComp
 $Comp
-L GND #PWR38
+L GND #PWR064
 U 1 1 52526592
 P 8300 5350
-F 0 "#PWR38" H 8300 5350 30  0001 C CNN
+F 0 "#PWR064" H 8300 5350 30  0001 C CNN
 F 1 "GND" H 8300 5280 30  0001 C CNN
 F 2 "" H 8300 5350 60  0000 C CNN
@@
 	2750 3650 950  3650
 Wire Wire Line
-	950  3550 950  3650
-Wire Wire Line
-	950  3650 950  3800
+	950  3550 950  3800
 Connection ~ 950  3650
 Wire Wire Line
@@
 	2950 4200 2950 4350
 Wire Wire Line
-	5950 1350 5950 1400
-Wire Wire Line
-	5950 1400 5950 2350
+	5950 1350 5950 2350
 Connection ~ 5950 1400
 Wire Wire Line
@@
 Connection ~ 9300 1850
 $Comp
-L VDD_PERIPH #U?
+L VDD_PERIPH #U065
 U 1 1 525D7AAA
 P 3150 6600
-F 0 "#U?" H 3150 6800 60  0001 C CNN
+F 0 "#U065" H 3150 6800 60  0001 C CNN
 F 1 "VDD_PERIPH" H 3150 6700 60  0000 C CNN
 F 2 "~" H 3150 6600 60  0000 C CNN
@@
 	1    0    0    -1
 $EndComp
+Wire Wire Line
+	7350 5700 7500 5700
+Wire Wire Line
+	7500 5700 7500 5300
+Wire Wire Line
+	6200 5700 6550 5700
 $EndSCHEMATC
