File: Hardware/WRFL_Launchpad.sch (KiCad schematic (older format))
At the start: 6 parts, among them P13 LAUNCHPAD_J1_J3, P14 LAUNCHPAD_J2_J4, P8 1x2_2.54_Fem, U11 REF3312

Commit message: 3d Kalman filter progress + minor sch
-moving towards a matrix (CMSIS) based kalman implementation
-cosmetic schematic  changes
Changed lines of the file:
@@
-EESchema Schematic File Version 2  date 10/31/2013 11:19:55 PM
+EESchema Schematic File Version 2
 LIBS:power
 LIBS:device
@@
 LIBS:WRFL
 LIBS:WRFL-cache
-EELAYER 27 0
+EELAYER 24 0
 EELAYER END
 $Descr A4 11693 8268
@@
 NoConn ~ 5550 1650
 $Comp
-L VDD_MCU #U13
+L VDD_MCU #U041
 U 1 1 524B47E3
 P 5200 1100
-F 0 "#U13" H 5200 1300 60  0001 C CNN
+F 0 "#U041" H 5200 1300 60  0001 C CNN
 F 1 "VDD_MCU" H 5200 1200 60  0000 C CNN
 F 2 "~" H 5200 1100 60  0000 C CNN
@@
 $EndComp
 $Comp
-L VDD_MCU #U11
+L VDD_MCU #U042
 U 1 1 525246DC
 P 1150 900
-F 0 "#U11" H 1150 1100 60  0001 C CNN
+F 0 "#U042" H 1150 1100 60  0001 C CNN
 F 1 "VDD_MCU" H 1150 1000 60  0000 C CNN
 F 2 "~" H 1150 900 60  0000 C CNN
@@
 $EndComp
 $Comp
-L GND #PWR29
+L GND #PWR043
 U 1 1 525246FA
 P 1800 1750
-F 0 "#PWR29" H 1800 1750 30  0001 C CNN
+F 0 "#PWR043" H 1800 1750 30  0001 C CNN
 F 1 "GND" H 1800 1680 30  0001 C CNN
 F 2 "" H 1800 1750 60  0000 C CNN
@@
 $EndComp
 $Comp
-L GND #PWR30
+L GND #PWR044
 U 1 1 52524709
 P 2650 1850
-F 0 "#PWR30" H 2650 1850 30  0001 C CNN
+F 0 "#PWR044" H 2650 1850 30  0001 C CNN
 F 1 "GND" H 2650 1780 30  0001 C CNN
 F 2 "" H 2650 1850 60  0000 C CNN
@@
 $EndComp
 Wire Wire Line
-	1150 1100 1150 1250
-Wire Wire Line
-	1150 1250 1150 1450
+	1150 1100 1150 1450
 Wire Wire Line
 	1150 1850 1150 1950
@@
 	1800 1600 1800 1750
 Wire Wire Line
-	2200 1250 2650 1250
-Wire Wire Line
-	2650 1250 3150 1250
+	2200 1250 3150 1250
 Wire Wire Line
 	2650 1250 2650 1350
@@
 VREF_SENS
 $Comp
-L VBUS #U12
+L VBUS #U045
 U 1 1 526426B1
 P 4300 3600
-F 0 "#U12" H 4300 3800 60  0001 C CNN
+F 0 "#U045" H 4300 3800 60  0001 C CNN
 F 1 "VBUS" H 4300 3700 60  0000 C CNN
 F 2 "~" H 4300 3600 60  0000 C CNN
@@
 	4300 3950 4300 3800
 $Comp
-L GND #PWR31
+L GND #PWR046
 U 1 1 52642A59
 P 4300 4200
-F 0 "#PWR31" H 4300 4200 30  0001 C CNN
+F 0 "#PWR046" H 4300 4200 30  0001 C CNN
 F 1 "GND" H 4300 4130 30  0001 C CNN
 F 2 "" H 4300 4200 60  0000 C CNN
@@
 $EndComp
 Wire Wire Line
-	3850 4150 4300 4150
-Wire Wire Line
-	4300 4150 4600 4150
+	3850 4150 4600 4150
 Wire Wire Line
 	4300 4150 4300 4200
@@
 	9900 5150 9300 5150
 $Comp
-L GND #PWR32
+L GND #PWR047
 U 1 1 52642B7B
 P 9600 4000
-F 0 "#PWR32" H 9600 4000 30  0001 C CNN
+F 0 "#PWR047" H 9600 4000 30  0001 C CNN
 F 1 "GND" H 9600 3930 30  0001 C CNN
 F 2 "" H 9600 4000 60  0000 C CNN
@@
 	9900 5750 9300 5750
 $Comp
-L GND #PWR28
+L GND #PWR048
 U 1 1 52664487
 P 1150 1950
-F 0 "#PWR28" H 1150 1950 30  0001 C CNN
+F 0 "#PWR048" H 1150 1950 30  0001 C CNN
 F 1 "GND" H 1150 1880 30  0001 C CNN
 F 2 "" H 1150 1950 60  0000 C CNN
@@
 $EndComp
 $Comp
-L PWR_FLAG #FLG3
+L PWR_FLAG #FLG049
 U 1 1 52665EE1
 P 4600 4000
-F 0 "#FLG3" H 4600 4095 30  0001 C CNN
+F 0 "#FLG049" H 4600 4095 30  0001 C CNN
 F 1 "PWR_FLAG" H 4600 4180 30  0000 C CNN
 F 2 "" H 4600 4000 60  0000 C CNN
